File: DBM/DBM.kicad_pcb (KiCad board)
At the start: 2 copper layers, 44 x 44 mm, 19 parts, among them J1 LO, J2 RF, J3 IF, T1 T_3743, T2 T_3743

Commit message: 准备打样
Parts:
- removed D5, D6, D7, D8: 1N60, cnsit:SMT_DIODE
- added H1: MountingHole, MountingHole:MountingHole_3.2mm_M3, F.Cu at (54.9, 49.3)
- added H2: MountingHole, MountingHole:MountingHole_3.2mm_M3, F.Cu at (85.9, 49.3)
- moved J1 9.50 mm to (67.1, 61.0)
- moved C1 8.71 mm to (67.1, 54.4), turned to 270 degrees
- moved R3 8.44 mm to (70.6, 48.8)
- moved R1 8.09 mm to (70.6, 51.8)
- moved R2 7.76 mm to (67.1, 49.8)
- moved T1 6.02 mm to (70.1, 43.7), turned to 270 degrees
- moved D2 3.35 mm to (75.7, 35.6)
- moved T2 3.28 mm to (70.1, 30.0)
- moved D4 3.25 mm to (65.0, 35.6)
- moved C2 1.02 mm to (80.8, 27.4)
- moved C3 0.71 mm to (59.4, 27.4)
Connections:
- D3 pad 1: Net-(D3-Pad1) -> Net-(D1-Pad2)
- D4 pad 2: Net-(D4-Pad2) -> Net-(D2-Pad1)
- T1 pad 3: Net-(D5-Pad2) -> Net-(D1-Pad2)
- T1 pad 6: Net-(D7-Pad1) -> Net-(D2-Pad1)
Routing:
- net Net-(D7-Pad1): track 17.4 -> 0.00 mm
- net Net-(D5-Pad2): track 15.5 -> 0.00 mm
- net Net-(D3-Pad1): track 8.37 -> 0.00 mm
- net Net-(D4-Pad2): track 8.37 -> 0.00 mm
- net Net-(D3-Pad2): track 17.6 -> 10.7 mm
- net Net-(D1-Pad1): track 15.5 -> 10.3 mm
- net Net-(D2-Pad1): track 8.44 -> 12.1 mm
- net Net-(R2-Pad1): track 7.57 -> 4.30 mm
- net Net-(C2-Pad1): track 9.73 -> 6.72 mm
- net Net-(C1-Pad2): track 8.08 -> 5.64 mm
- net Net-(D1-Pad2): track 8.37 -> 6.90 mm
- net Net-(C3-Pad2): track 14.0 -> 13.0 mm
- net Net-(C1-Pad1): track 6.23 -> 5.23 mm
- net Net-(C2-Pad2): track 10.2 -> 9.30 mm
- net Net-(C3-Pad1): track 10.1 -> 9.38 mm
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- added copper zone on B.Cu, net GNDA
- added copper zone on F.Cu, net GNDA
Other:
- board text added: "30mm"
